File: kicad/feed-selector-v2.kicad_sch (KiCad schematic)
At the start: 11 parts, among them J1 CREEP/RAPID, J2 512C, J3 POT, J4 UART, SW1 CLEAR_EEPROM, U1 MCP41HV51-103E/ST

Commit message: documentation
Other:
- title: (none) -> MAHO MH300M Feed Controller
Changed lines of the file:
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@@
 	(generator_version "8.0")
 	(paper "A5")
+	(title_block
+		(title "MAHO MH300M Feed Controller")
+		(rev "20240822-r1")
+	)
 	(junction
 		(at 25.4 90.17)
@@
 		)
 	)
-	(text_box "10mA max"
+	(text_box "5mA max"
 		(exclude_from_sim no)
 		(at 76.2 130.81 0)
